Commit message: Modified paths to meshes

File: iq_sim/urdf/iris_urdf.urdf (robot description, URDF)
Before this commit: robot iris_demo, 6 links, 5 joints
Links:
- link iris_demo__hokuyo_link: geometry collision box size=0.08 0.08 0.08; visual mesh filename=package://iq_sim/models/hokuyo/meshes/hokuyo.dae scale=1.0 1.0 1.0
- link iris_demo__iris__base_link: geometry collision box size=1 1 1; visual mesh filename=package://iq_sim/models/iris_with_standoffs/meshes/iris.dae scale=1.0 1.0 1.0
